File: mainBoardV2/mainBoardV2.kicad_pcb (KiCad board)
At the start: 2 copper layers, 32 parts, among them J1 USB4125-GF-A_REVA2, U1 ESP32-CAM, U2 ESP32-DEVKITC-32E, U3 MCP73871-2AAI_ML, U4 MPU6050_Module, U5 TPS61090RSARG4

Commit message: Update mainBoardV2.kicad_pcb
Other:
- board text added: "This is a test"
Changed lines of the file:
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@@
+		)
+	)
+	(gr_text "This is a test"
+		(at 178 140.5 0)
+		(layer "Cmts.User")
+		(effects
+			(font
+				(size 1.5 1.5)
+				(thickness 0.3)
+				(bold yes)
+			)
+			(justify left bottom)
 		)
 	)

Commit message: 2.28.26.C1
Parts:
- U7: footprint APGF1012GBRC-07:LED_APGF1012GBRC-07 -> LED_SMD:BivarSMTL-SRGY
- moved U7 249.7 mm to (248.5, 36.4)
Connections:
- R9 pad 1: Net-(U7-Blue) -> Net-(U7-Yellow)
- U7 pad 2: Net-(U7-Red) -> Net-(U7-Yellow)
- U7 pad 3: +5V -> Net-(U7-Red)
- U7 pad 4: Net-(U7-Blue) -> +5V
Other:
- board text removed: "This is a test"
Changed lines of the file:
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@@
 	(net 66 "Net-(U5-FB)")
 	(net 67 "Net-(U7-Green)")
-	(net 68 "Net-(U7-Blue)")
+	(net 68 "Net-(U7-Yellow)")
 	(net 69 "Net-(RintoGyro1-Pad1)")
 	(net 70 "unconnected-(U4-PadINT)")
@@
 		)
 	)
-	(footprint "APGF1012GBRC-07:LED_APGF1012GBRC-07"
-		(layer "F.Cu")
-		(at 1.375 0.8)
-		(property "Reference" "U7"
-			(at 2.4 -2.41 0)
-			(layer "F.SilkS")
-			(effects
-				(font
-					(size 1 1)
-					(thickness 0.15)
-				)
-			)
-		)
-		(property "Value" "~"
-			(at 11.29 2.41 0)
-			(layer "F.Fab")
-			(effects
-				(font
-					(size 1 1)
-					(thickness 0.15)
-				)
-			)
-		)
-		(property "Datasheet" ""
-			(at 0 0 0)
-			(layer "F.Fab")
-			(hide yes)
-			(effects
-				(font
-					(size 1.27 1.27)
-					(thickness 0.15)
-				)
-			)
-		)
-		(property "Description" ""
-			(at 0 0 0)
-			(layer "F.Fab")
-			(hide yes)
-			(effects
-				(font
-					(size 1.27 1.27)
-					(thickness 0.15)
-				)
-			)
-		)
-		(sheetname "/")
-		(sheetfile "mainBoardV2.kicad_sch")
-		(attr smd)
-		(fp_poly
-			(pts
-				(xy -0.575 -0.575) (xy -0.075 -0.575) (xy -0.075 -0.075) (xy -0.575 -0.075)
-			)
-			(stroke
-				(width 0.01)
-				(type solid)
-			)
-			(fill yes)
-			(layer "F.Mask")
-		)
-		(fp_poly
-			(pts
-				(xy -0.575 0.075) (xy -0.075 0.075) (xy -0.075 0.575) (xy -0.575 0.575)
-			)
-			(stroke
-				(width 0.01)
-				(type solid)
-			)
-			(fill yes)
-			(layer "F.Mask")
-		)
-		(fp_poly
-			(pts
-				(xy 0.075 -0.575) (xy 0.575 -0.575) (xy 0.575 -0.075) (xy 0.075 -0.075)
-			)
-			(stroke
-				(width 0.01)
-				(type solid)
-			)
-			(fill yes)
-			(layer "F.Mask")
-		)
-		(fp_poly
-			(pts
-				(xy 0.075 0.075) (xy 0.575 0.075) (xy 0.575 0.575) (xy 0.075 0.575)
-			)
-			(stroke
-				(width 0.01)
-				(type solid)
-			)
-			(fill yes)
-			(layer "F.Mask")
-		)
-		(fp_circle
-			(center -1.175 -0.325)
-			(end -1.075 -0.325)
-			(stroke
-				(width 0.2)
-				(type solid)
-			)
-			(fill no)
-			(layer "F.SilkS")
-		)
-		(fp_line
-			(start -0.775 -0.775)
-			(end -0.775 0.775)
-			(stroke
-				(width 0.05)
-				(type solid)
-			)
-			(layer "F.CrtYd")
-		)
-		(fp_line
-			(start -0.775 0.775)
-			(end 0.775 0.775)
-			(stroke
-				(width 0.05)
-				(type solid)
-			)
-			(layer "F.CrtYd")
-		)
-		(fp_line
-			(start 0.775 -0.775)
-			(end -0.775 -0.775)
-			(stroke
-				(width 0.05)
-				(type solid)
-			)
-			(layer "F.CrtYd")
-		)
-		(fp_line
-			(start 0.775 0.775)
-			(end 0.775 -0.775)
-			(stroke
-				(width 0.05)
-				(type solid)
-			)
-			(layer "F.CrtYd")
-		)
-		(fp_line
-			(start -0.5 -0.5)
-			(end 0.5 -0.5)
-			(stroke
-				(width 0.127)
-				(type solid)
-			)
-			(layer "F.Fab")
-		)
-		(fp_line
-			(start -0.5 0.5)
-			(end -0.5 -0.5)
-			(stroke
-				(width 0.127)
-				(type solid)
-			)
-			(layer "F.Fab")
-		)
-		(fp_line
-			(start 0.5 -0.5)
-			(end 0.5 0.5)
-			(stroke
-				(width 0.127)
-				(type solid)
-			)
-			(layer "F.Fab")
-		)
-		(fp_line
-			(start 0.5 0.5)
-			(end -0.5 0.5)
-			(stroke
-				(width 0.127)
-				(type solid)
-			)
-			(layer "F.Fab")
-		)
-		(fp_circle
-			(center -1.175 -0.325)
-			(end -1.075 -0.325)
-			(stroke
-				(width 0.2)
-				(type solid)
-			)
-			(fill no)
-			(layer "F.Fab")
-		)
-		(pad "1" smd rect
-			(at -0.325 -0.325)
-			(size 0.4 0.4)
-			(layers "F.Cu" "F.Paste")
-			(net 67 "Net-(U7-Green)")
-			(pinfunction "Green")
-			(pintype "bidirectional")
-		)
-		(pad "2" smd rect
-			(at -0.325 0.325)
-			(size 0.4 0.4)
-			(layers "F.Cu" "F.Paste")
-			(net 74 "Net-(U7-Red)")
-			(pinfunction "Red")
-			(pintype "bidirectional")
-		)
-		(pad "3" smd rect
-			(at 0.325 0.325)
-			(size 0.4 0.4)
-			(layers "F.Cu" "F.Paste")
-			(net 2 "+5V")
-			(pinfunction "Polarity_Marker")
-			(pintype "bidirectional")
-		)
-		(pad "4" smd rect
-			(at 0.325 -0.325)
-			(size 0.4 0.4)
-			(layers "F.Cu" "F.Paste")
-			(net 68 "Net-(U7-Blue)")
-			(pinfunction "Blue")
-			(pintype "bidirectional")
-		)
-		(embedded_fonts no)
-	)
 	(footprint "T495C107K006ATE150(1):CAPMP6032X250"
 		(layer "F.Cu")
@@
 		(embedded_fonts no)
 	)
+	(footprint "LED_SMD:BivarSMTL-SRGY"
+		(layer "F.Cu")
+		(at 248.5 36.4)
+		(property "Reference" "U7"
+			(at -0.12 8.52 0)
+			(unlocked yes)
+			(layer "F.SilkS")
+			(effects
+				(font
+					(size 1 1)
+					(thickness 0.1)
+				)
+			)
+		)
+		(property "Value" "~"
+			(at 0.04 12.87 0)
+			(unlocked yes)
+			(layer "F.Fab")
+			(effects
+				(font
+					(size 1 1)
+					(thickness 0.15)
+				)
+			)
+		)
+		(property "Datasheet" ""
+			(at 0 0 0)
+			(unlocked yes)
+			(layer "F.Fab")
+			(hide yes)
+			(effects
+				(font
+					(size 1 1)
+					(thickness 0.15)
+				)
+			)
+		)
+		(property "Description" ""
+			(at 0 0 0)
+			(unlocked yes)
+			(layer "F.Fab")
+			(hide yes)
+			(effects
+				(font
+					(size 1 1)
+					(thickness 0.15)
+				)
+			)
+		)
+		(sheetname "/")
+		(sheetfile "mainBoardV2.kicad_sch")
+		(attr smd)
+		(fp_line
+			(start -0.66 -0.15)
+			(end -0.66 3.05)
+			(stroke
+				(width 0.1)
+				(type default)
+			)
+			(layer "F.SilkS")
+		)
+		(fp_line
+			(start 2.14 -0.15)
+			(end 2.14 3.05)
+			(stroke
+				(width 0.1)
+				(type default)
+			)
+			(layer "F.SilkS")
+		)
+		(fp_circle
+			(center 2.59 -1.11)
+			(end 2.66 -0.97)
+			(stroke
+				(width 0.1)
+				(type solid)
+			)
+			(fill yes)
+			(layer "F.SilkS")
+		)
+		(fp_text user "${REFERENCE}"
+			(at 0.04 10.66 0)
+			(unlocked yes)
+			(layer "F.Fab")
+			(effects
+				(font
+					(size 1 1)
+					(thickness 0.15)
+				)
+			)
+		)
+		(pad "1" smd roundrect
+			(at 0 0)
+			(size 0.9 1.5)
+			(layers "F.Cu" "F.Mask" "F.Paste")
+			(roundrect_rratio 0.15)
+			(net 67 "Net-(U7-Green)")
+			(pinfunction "Green")
+			(pintype "bidirectional")
+		)
+		(pad "2" smd roundrect
+			(at 0 3.1)
+			(size 0.9 1.5)
+			(layers "F.Cu" "F.Mask" "F.Paste")
+			(roundrect_rratio 0.15)
+			(net 68 "Net-(U7-Yellow)")
+			(pinfunction "Yellow")
+			(pintype "bidirectional")
+		)
+		(pad "3" smd roundrect
+			(at 1.5 0)
+			(size 0.9 1.5)
+			(layers "F.Cu" "F.Mask" "F.Paste")
+			(roundrect_rratio 0.15)
+			(net 74 "Net-(U7-Red)")
+			(pinfunction "Red")
+			(pintype "bidirectional")
+		)
+		(pad "4" smd roundrect
+			(at 1.5 3.1)
+			(size 0.9 1.5)
+			(layers "F.Cu" "F.Mask" "F.Paste")
+			(roundrect_rratio 0.15)
+			(net 2 "+5V")
+			(pinfunction "Common_Anode")
+			(pintype "bidirectional")
+		)
+		(embedded_fonts no)
+	)
 	(footprint "USB4125-GF-A_REVA2:GCT_USB4125-GF-A_REVA2"
 		(layer "F.Cu")
@@
 			(layers "F.Cu" "F.Mask" "F.Paste")
 			(roundrect_rratio 0.208333)
-			(net 68 "Net-(U7-Blue)")
+			(net 68 "Net-(U7-Yellow)")
 			(pintype "passive")
 		)
@@
 		)
 	)
-	(gr_text "This is a test"
-		(at 178 140.5 0)
-		(layer "Cmts.User")
-		(effects
-			(font
-				(size 1.5 1.5)
-				(thickness 0.3)
-				(bold yes)
-			)
-			(justify left bottom)
-		)
-	)

Commit message: 2.28.28.C2
Parts:
- moved J1 169.4 mm to (208.2, 39.3)
- moved R15 163.2 mm to (192.0, 45.0)
- moved R14 157.9 mm to (196.5, 41.5)
- moved C5 108.1 mm to (262.0, 35.0)
- moved C4 105.1 mm to (251.5, 24.0)
- moved C6 91.0 mm to (255.5, 48.0)
- moved C2 50.5 mm to (265.0, 87.0)
- moved C1 49.7 mm to (271.5, 86.5)
- moved R9 34.1 mm to (227.0, 47.0)
- moved R6 33.2 mm to (222.5, 35.0)
- moved C3 31.8 mm to (267.0, 94.0)
- moved R10 25.0 mm to (226.0, 52.0)
- moved R11 24.4 mm to (249.5, 38.5)
- moved U7 15.6 mm to (236.0, 45.7)
- moved R12 13.1 mm to (250.0, 43.5)
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Routing:
- added copper zone on B.Cu, net GND
Changed lines of the file:
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@@
 	(footprint "Capacitor_SMD:C_0805_2012Metric_Pad1.18x1.45mm_HandSolder"
 		(layer "F.Cu")
-		(at 254 133)
+		(at 271.5 86.5)
 		(descr "Capacitor SMD 0805 (2012 Metric), square (rectangular) end terminal, IPC-7351 nominal with elongated pad for handsoldering. (Body size source: IPC-SM-782 page 76, https://www.pcb-3d.com/wordpress/wp-content/uploads/ipc-sm-782a_amendment_1_and_2.pdf, https://docs.google.com/spreadsheets/d/1BsfQQcO9C6DZCsRaXUlFlo91Tg2WpOkGARC1WS5S8t0/edit?usp=sharing), generated with kicad-footprint-generator")
 		(tags "capacitor handsolder")
@@
 	(footprint "T495C107K006ATE150(1):CAPMP6032X250"
 		(layer "F.Cu")
-		(at 263 125.5)
+		(at 267 94)
 		(property "Reference" "C3"
 			(at -1.36612 -3.04249 0)
@@
 	(footprint "Resistor_SMD:R_0805_2012Metric_Pad1.20x1.40mm_HandSolder"
 		(layer "F.Cu")
-		(at 225.5 46)
+		(at 232 47)
 		(descr "Resistor SMD 0805 (2012 Metric), square (rectangular) end terminal, IPC-7351 nominal with elongated pad for handsoldering. (Body size source: IPC-SM-782 page 72, https://www.pcb-3d.com/wordpress/wp-content/uploads/ipc-sm-782a_amendment_1_and_2.pdf), generated with kicad-footprint-generator")
 		(tags "resistor handsolder")
@@
 	(footprint "Resistor_SMD:R_0805_2012Metric_Pad1.20x1.40mm_HandSolder"
 		(layer "F.Cu")
-		(at 254.5 26)
+		(at 222.5 35)
 		(descr "Resistor SMD 0805 (2012 Metric), square (rectangular) end terminal, IPC-7351 nominal with elongated pad for handsoldering. (Body size source: IPC-SM-782 page 72, https://www.pcb-3d.com/wordpress/wp-content/uploads/ipc-sm-782a_amendment_1_and_2.pdf), generated with kicad-footprint-generator")
 		(tags "resistor handsolder")
@@
 	(footprint "Capacitor_SMD:C_0805_2012Metric_Pad1.18x1.45mm_HandSolder"
 		(layer "F.Cu")
-		(at 266.9625 143)
+		(at 262 35)
 		(descr "Capacitor SMD 0805 (2012 Metric), square (rectangular) end terminal, IPC-7351 nominal with elongated pad for handsoldering. (Body size source: IPC-SM-782 page 76, https://www.pcb-3d.com/wordpress/wp-content/uploads/ipc-sm-782a_amendment_1_and_2.pdf, https://docs.google.com/spreadsheets/d/1BsfQQcO9C6DZCsRaXUlFlo91Tg2WpOkGARC1WS5S8t0/edit?usp=sharing), generated with kicad-footprint-generator")
 		(tags "capacitor handsolder")
@@
 	(footprint "Resistor_SMD:R_0805_2012Metric_Pad1.20x1.40mm_HandSolder"
 		(layer "F.Cu")
-		(at 231.5 55)
+		(at 249.5 38.5)
 		(descr "Resistor SMD 0805 (2012 Metric), square (rectangular) end terminal, IPC-7351 nominal with elongated pad for handsoldering. (Body size source: IPC-SM-782 page 72, https://www.pcb-3d.com/wordpress/wp-content/uploads/ipc-sm-782a_amendment_1_and_2.pdf), generated with kicad-footprint-generator")
 		(tags "resistor handsolder")
@@
 	(footprint "Resistor_SMD:R_0805_2012Metric_Pad1.20x1.40mm_HandSolder"
 		(layer "F.Cu")
-		(at 46.5 119)
+		(at 192 45)
 		(descr "Resistor SMD 0805 (2012 Metric), square (rectangular) end terminal, IPC-7351 nominal with elongated pad for handsoldering. (Body size source: IPC-SM-782 page 72, https://www.pcb-3d.com/wordpress/wp-content/uploads/ipc-sm-782a_amendment_1_and_2.pdf), generated with kicad-footprint-generator")
 		(tags "resistor handsolder")
@@
 	(footprint "TPS61090RSARG4:QFN65P400X400X100-17N"
 		(layer "F.Cu")
-		(at 249 103)
+		(at 248.955 103)
 		(property "Reference" "U5"
 			(at 0.005395 -3.794595 0)
@@
 	(footprint "Resistor_SMD:R_0805_2012Metric_Pad1.20x1.40mm_HandSolder"
 		(layer "F.Cu")
-		(at 239.5 96)
+		(at 237.5 96)
 		(descr "Resistor SMD 0805 (2012 Metric), square (rectangular) end terminal, IPC-7351 nominal with elongated pad for handsoldering. (Body size source: IPC-SM-782 page 72, https://www.pcb-3d.com/wordpress/wp-content/uploads/ipc-sm-782a_amendment_1_and_2.pdf), generated with kicad-footprint-generator")
 		(tags "resistor handsolder")
@@
 	(footprint "Capacitor_SMD:C_0805_2012Metric_Pad1.18x1.45mm_HandSolder"
 		(layer "F.Cu")
-		(at 276.9625 126)
+		(at 251.4625 24)
 		(descr "Capacitor SMD 0805 (2012 Metric), square (rectangular) end terminal, IPC-7351 nominal with elongated pad for handsoldering. (Body size source: IPC-SM-782 page 76, https://www.pcb-3d.com/wordpress/wp-content/uploads/ipc-sm-782a_amendment_1_and_2.pdf, https://docs.google.com/spreadsheets/d/1BsfQQcO9C6DZCsRaXUlFlo91Tg2WpOkGARC1WS5S8t0/edit?usp=sharing), generated with kicad-footprint-generator")
 		(tags "capacitor handsolder")
@@
 	(footprint "Inductor_SMD:Sumida_senior"
 		(layer "F.Cu")
-		(at 236.095 113.985)
+		(at 239.095 113.985)
 		(property "Reference" "L1"
 			(at 5.36 14.88 0)
@@
 	(footprint "LED_SMD:BivarSMTL-SRGY"
 		(layer "F.Cu")
-		(at 248.5 36.4)
+		(at 235.956738 45.733263)
 		(property "Reference" "U7"
-			(at -0.12 8.52 0)
+			(at 0.543262 5.266737 0)
 			(unlocked yes)
 			(layer "F.SilkS")
@@
 			(unlocked yes)
 			(layer "F.Fab")
+			(hide yes)
 			(effects
 				(font
@@
 			(layer "F.SilkS")
 		)
-		(fp_text user "${REFERENCE}"
-			(at 0.04 10.66 0)
-			(unlocked yes)
-			(layer "F.Fab")
-			(effects
-				(font
-					(size 1 1)
-					(thickness 0.15)
-				)
-			)
-		)
 		(pad "1" smd roundrect
 			(at 0 0)
@@
 	(footprint "USB4125-GF-A_REVA2:GCT_USB4125-GF-A_REVA2"
 		(layer "F.Cu")
-		(at 49.5 98.5 90)
+		(at 208.2 39.32 90)
 		(property "Reference" "J1"
 			(at -0.125 -5.135 90)
@@
 	(footprint "Resistor_SMD:R_0805_2012Metric_Pad1.20x1.40mm_HandSolder"
 		(layer "F.Cu")
-		(at 221 27.5)
+		(at 226 52)
 		(descr "Resistor SMD 0805 (2012 Metric), square (rectangular) end terminal, IPC-7351 nominal with elongated pad for handsoldering. (Body size source: IPC-SM-782 page 72, https://www.pcb-3d.com/wordpress/wp-content/uploads/ipc-sm-782a_amendment_1_and_2.pdf), generated with kicad-footprint-generator")
 		(tags "resistor handsolder")
@@
 	(footprint "Resistor_SMD:R_0805_2012Metric_Pad1.20x1.40mm_HandSolder"
 		(layer "F.Cu")
-		(at 256.5 43.5)
+		(at 255.5 40.5)
 		(descr "Resistor SMD 0805 (2012 Metric), square (rectangular) end terminal, IPC-7351 nominal with elongated pad for handsoldering. (Body size source: IPC-SM-782 page 72, https://www.pcb-3d.com/wordpress/wp-content/uploads/ipc-sm-782a_amendment_1_and_2.pdf), generated with kicad-footprint-generator")
 		(tags "resistor handsolder")
@@
 	(footprint "Resistor_SMD:R_0805_2012Metric_Pad1.20x1.40mm_HandSolder"
 		(layer "F.Cu")
-		(at 246 56)
+		(at 250 43.5)
 		(descr "Resistor SMD 0805 (2012 Metric), square (rectangular) end terminal, IPC-7351 nominal with elongated pad for handsoldering. (Body size source: IPC-SM-782 page 72, https://www.pcb-3d.com/wordpress/wp-content/uploads/ipc-sm-782a_amendment_1_and_2.pdf), generated with kicad-footprint-generator")
 		(tags "resistor handsolder")
@@
 	(footprint "Resistor_SMD:R_0805_2012Metric_Pad1.20x1.40mm_HandSolder"
 		(layer "F.Cu")
-		(at 260 55.5)
+		(at 227 47)
 		(descr "Resistor SMD 0805 (2012 Metric), square (rectangular) end terminal, IPC-7351 nominal with elongated pad for handsoldering. (Body size source: IPC-SM-782 page 72, https://www.pcb-3d.com/wordpress/wp-content/uploads/ipc-sm-782a_amendment_1_and_2.pdf), generated with kicad-footprint-generator")
 		(tags "resistor handsolder")
@@
 	(footprint "Resistor_SMD:R_0805_2012Metric_Pad1.20x1.40mm_HandSolder"
 		(layer "F.Cu")
-		(at 56 113.5)
+		(at 196.5 41.5)
 		(descr "Resistor SMD 0805 (2012 Metric), square (rectangular) end terminal, IPC-7351 nominal with elongated pad for handsoldering. (Body size source: IPC-SM-782 page 72, https://www.pcb-3d.com/wordpress/wp-content/uploads/ipc-sm-782a_amendment_1_and_2.pdf), generated with kicad-footprint-generator")
 		(tags "resistor handsolder")
@@
 	(footprint "Capacitor_SMD:C_0805_2012Metric_Pad1.18x1.45mm_HandSolder"
 		(layer "F.Cu")
-		(at 254 139)
+		(at 255.5 48)
 		(descr "Capacitor SMD 0805 (2012 Metric), square (rectangular) end terminal, IPC-7351 nominal with elongated pad for handsoldering. (Body size source: IPC-SM-782 page 76, https://www.pcb-3d.com/wordpress/wp-content/uploads/ipc-sm-782a_amendment_1_and_2.pdf, https://docs.google.com/spreadsheets/d/1BsfQQcO9C6DZCsRaXUlFlo91Tg2WpOkGARC1WS5S8t0/edit?usp=sharing), generated with kicad-footprint-generator")
 		(tags "capacitor handsolder")
@@
 	(footprint "Capacitor_SMD:C_0805_2012Metric_Pad1.18x1.45mm_HandSolder"
 		(layer "F.Cu")
-		(at 277.0375 136)
+		(at 265 87)
 		(descr "Capacitor SMD 0805 (2012 Metric), square (rectangular) end terminal, IPC-7351 nominal with elongated pad for handsoldering. (Body size source: IPC-SM-782 page 76, https://www.pcb-3d.com/wordpress/wp-content/uploads/ipc-sm-782a_amendment_1_and_2.pdf, https://docs.google.com/spreadsheets/d/1BsfQQcO9C6DZCsRaXUlFlo91Tg2WpOkGARC1WS5S8t0/edit?usp=sharing), generated with kicad-footprint-generator")
 		(tags "capacitor handsolder")
@@
 	(footprint "Resistor_SMD:R_0805_2012Metric_Pad1.20x1.40mm_HandSolder"
 		(layer "F.Cu")
-		(at 268 100.5)
+		(at 263 110)
 		(descr "Resistor SMD 0805 (2012 Metric), square (rectangular) end terminal, IPC-7351 nominal with elongated pad for handsoldering. (Body size source: IPC-SM-782 page 72, https://www.pcb-3d.com/wordpress/wp-content/uploads/ipc-sm-782a_amendment_1_and_2.pdf), generated with kicad-footprint-generator")
 		(tags "resistor handsolder")
@@
 			)
 		)
+	)
+	(zone
+		(net 4)
+		(net_name "GND")
+		(layer "B.Cu")
+		(hatch edge 0.5)
+		(connect_pads
+			(clearance 0)
+		)
+		(min_thickness 0.25)
+		(filled_areas_thickness no)
+		(fill yes
+			(thermal_gap 0.5)
+			(thermal_bridge_width 0.5)
+		)
+		(polygon
+			(pts
+				(xy 12 12) (xy 285 12) (xy 285 166) (xy 12 165.5)
+			)
+		)

Commit message: 2.28.26.C3
Parts:
- moved U6 146.9 mm to (236.5, 22.2), turned to 0 degrees
- moved L1 135.5 mm to (352.6, 40.0)
- moved C1 135.5 mm to (385.0, 12.5)
- moved C2 135.5 mm to (378.5, 13.0)
- moved C3 135.5 mm to (380.5, 20.0)
- moved R1 135.5 mm to (351.0, 22.0)
- moved R2 135.5 mm to (348.0, 27.0)
- moved R3 135.5 mm to (376.5, 36.0)
- moved R4 135.5 mm to (371.5, 38.5)
- moved R5 135.5 mm to (365.5, 18.0)
- moved U5 135.5 mm to (362.5, 29.0)
- moved C6 25.3 mm to (237.5, 30.2)
- moved C5 24.5 mm to (237.7, 38.1)
- moved C4 20.7 mm to (233.7, 34.5), turned to -90 degrees
- moved U3 4.90 mm to (237.5, 34.0), turned to 90 degrees

Commit message: 2.28.26.C4
Parts:
- moved R13 37.1 mm to (219.5, 31.8), turned to 180 degrees
- moved R15 28.6 mm to (212.6, 25.1)
- moved J1 25.7 mm to (222.2, 17.8), turned to 180 degrees
- moved R12 24.7 mm to (229.6, 29.5)
- moved R14 24.4 mm to (212.6, 23.1)
- moved R11 21.1 mm to (229.6, 31.5), turned to 180 degrees
- moved C5 20.1 mm to (219.5, 29.7), turned to 180 degrees
- moved R10 18.2 mm to (220.0, 34.8), turned to -90 degrees
- moved R8 14.6 mm to (224.0, 34.8), turned to -90 degrees
- moved U3 13.6 mm to (224.8, 29.0), turned to 0 degrees
- moved R9 13.2 mm to (222.0, 34.8), turned to -90 degrees
- moved U7 12.9 mm to (230.1, 34.3), turned to -90 degrees
- moved C4 12.4 mm to (225.6, 25.1), turned to 0 degrees
- moved R7 11.8 mm to (219.5, 27.7), turned to 180 degrees
- moved R6 9.90 mm to (221.5, 25.1), turned to 180 degrees
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
Commit message: 2.28.26.C5
Parts:
- removed U1: ESP32-CAM, ESP32-CAM:ESP32-CAM
- moved C1 242.8 mm to (153.2, 84.6)
- moved C2 241.2 mm to (150.6, 91.9), turned to 180 degrees
- moved C3 235.3 mm to (156.9, 93.2)
- moved R3 233.3 mm to (150.6, 94.2)
- moved R4 228.3 mm to (150.6, 96.3), turned to 180 degrees
- moved R5 225.0 mm to (154.9, 97.3), turned to 180 degrees
- moved R1 218.4 mm to (142.2, 86.1), turned to 180 degrees
- moved U5 218.0 mm to (152.7, 88.1), turned to 180 degrees
- moved R2 214.8 mm to (142.2, 88.6)
- moved L1 200.5 mm to (156.0, 79.4)
- moved R14 117.0 mm to (110.5, 80.1)
- moved R15 117.0 mm to (110.5, 82.1)
- moved R9 117.0 mm to (119.9, 91.8)
- moved C4 117.0 mm to (123.4, 82.1)
- moved C5 117.0 mm to (117.3, 86.7)
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
Commit message: 3.1.26.C2
Have a preliminary layout, ready to perfect
Parts:
- added ?: , , F.Cu at (92.2, 73.4)
- added ?: , , F.Cu at (92.2, 71.1)
- moved L1 76.5 mm to (84.0, 105.1), turned to 90 degrees
- moved U6 72.8 mm to (91.5, 121.7), turned to 0 degrees
- moved C1 69.4 mm to (89.5, 112.3)
- moved C3 65.5 mm to (93.0, 107.6), turned to 180 degrees
- moved U5 63.5 mm to (94.1, 112.8), turned to -90 degrees
- moved RintoCam1 59.8 mm to (92.2, 67.8), turned to 90 degrees
- moved R1 59.2 mm to (92.1, 117.5), turned to 0 degrees
- moved R5 56.9 mm to (99.3, 109.4), turned to 0 degrees
- moved R4 55.2 mm to (98.5, 114.4)
- moved C2 55.1 mm to (96.9, 104.1), turned to 0 degrees
- moved R3 54.9 mm to (98.5, 111.7), turned to 180 degrees
- moved R2 54.6 mm to (95.9, 117.5), turned to 180 degrees
- moved J1 53.4 mm to (116.8, 125.0), turned to 0 degrees
- moved U4 50.6 mm to (125.9, 83.2)
- moved R14 46.1 mm to (124.7, 124.0)
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Routing:
- net GND: track 0.00 -> 216.8 mm, vias 0 -> 19
- net Net-(SW1-A): track 0.00 -> 129.0 mm, vias 0 -> 2
- net Net-(U2-IO17): track 0.00 -> 51.3 mm, vias 0 -> 2
- net Net-(U2-IO5): track 0.00 -> 47.0 mm, vias 0 -> 1
- net +5V: track 0.00 -> 32.0 mm, vias 0 -> 4
- net Net-(U3-VBAT_SENSE): track 0.00 -> 12.7 mm
- net Net-(U7-Green): track 0.00 -> 12.4 mm
- net Net-(U3-VPCC): track 0.00 -> 12.3 mm, vias 0 -> 2
- net Net-(U7-Yellow): track 0.00 -> 12.1 mm, vias 0 -> 2
- net Net-(U3-STAT2): track 0.00 -> 10.0 mm, vias 0 -> 2
- net Net-(U3-~{PG}): track 0.00 -> 9.41 mm
- net Net-(J1-CC1): track 0.00 -> 8.05 mm
- net Net-(J1-CC2): track 0.00 -> 7.91 mm
- net Net-(RintoGyro1-Pad1): track 0.00 -> 5.81 mm
- net Net-(U3-STAT1/*LBO): track 0.00 -> 4.83 mm
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- added copper zone on F.Cu, net (none)
- added copper zone on F.Cu, net +5V
- added copper zone on F.Cu, net Net-(SW1-A)
- removed copper zone on B.Cu, net GND
Other:
- board outline added: 55.9 x 117 mm
- board text added: "ON/OFF here"

Commit message: 3.1.26.C3
Done for the day?
Changed lines of the file:
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@@
 		(at 94.096744 112.760744 -90)
 		(property "Reference" "U5"
-			(at 8.651256 9.768744 0)
+			(at 11.684 -6.096 90)
 			(layer "F.SilkS")
 			(effects
